File: lipo_parallel_board/lipo_parallel_board.kicad_pcb (KiCad board)
At the start: 0 parts

Commit message: iniziato il pcb
Parts:
- added J1: Conn_01x07_Female, Connector_JST:JST_XH_B7B-XH-AM_1x07_P2.50mm_Vertical, F.Cu at (140.6, 46.1)
- added J10: Conn_01x03_Female, Connector_JST:JST_XH_B3B-XH-AM_1x03_P2.50mm_Vertical, F.Cu at (176.5, 65.2)
- added J11: Conn_01x03_Female, Connector_JST:JST_XH_B3B-XH-AM_1x03_P2.50mm_Vertical, F.Cu at (177.9, 95.0)
- added J12: XT30_F, Connector_AMASS:AMASS_XT30U-F_1x02_P5.0mm_Vertical, F.Cu at (125.7, 130.2)
- added J13: XT60_F, Connector_AMASS:AMASS_XT60-F_1x02_P7.20mm_Vertical, F.Cu at (122.0, 120.2)
- added J14: XT30_F, Connector_AMASS:AMASS_XT30U-F_1x02_P5.0mm_Vertical, F.Cu at (125.7, 104.7)
- added J15: XT60_F, Connector_AMASS:AMASS_XT60-F_1x02_P7.20mm_Vertical, F.Cu at (144.6, 91.8)
- added J16: Conn_01x05_Female, Connector_JST:JST_XH_B5B-XH-AM_1x05_P2.50mm_Vertical, F.Cu at (176.0, 73.6)
- added J17: Conn_01x05_Female, Connector_JST:JST_XH_B5B-XH-AM_1x05_P2.50mm_Vertical, F.Cu at (97.8, 97.8)
- added J18: XT30_F, Connector_AMASS:AMASS_XT30U-F_1x02_P5.0mm_Vertical, F.Cu at (125.7, 77.6)
- added J19: XT60_F, Connector_AMASS:AMASS_XT60-F_1x02_P7.20mm_Vertical, F.Cu at (144.5, 71.3)
- added J2: Conn_01x03_Female, Connector_JST:JST_XH_B3B-XH-AM_1x03_P2.50mm_Vertical, F.Cu at (178.3, 126.3)
- added J20: XT30_F, Connector_AMASS:AMASS_XT30U-F_1x02_P5.0mm_Vertical, F.Cu at (148.3, 101.8)
- added J21: XT60_F, Connector_AMASS:AMASS_XT60-F_1x02_P7.20mm_Vertical, F.Cu at (122.0, 94.7)
- added J22: Conn_01x07_Female, Connector_JST:JST_XH_B7B-XH-AM_1x07_P2.50mm_Vertical, F.Cu at (177.7, 144.9)
- added J23: Conn_01x07_Female, Connector_JST:JST_XH_B7B-XH-AM_1x07_P2.50mm_Vertical, F.Cu at (176.4, 83.7)
- added J24: XT30_F, Connector_AMASS:AMASS_XT30U-F_1x02_P5.0mm_Vertical, F.Cu at (149.6, 138.7)
- added J25: XT60_F, Connector_AMASS:AMASS_XT60-F_1x02_P7.20mm_Vertical, F.Cu at (122.0, 68.2)
- added J26: Conn_01x03_Female, Connector_JST:JST_XH_B3B-XH-AM_1x03_P2.50mm_Vertical, F.Cu at (97.8, 116.7)
- added J27: Conn_01x03_Female, Connector_JST:JST_XH_B3B-XH-AM_1x03_P2.50mm_Vertical, F.Cu at (97.8, 90.7)
- added J28: XT30_F, Connector_AMASS:AMASS_XT30U-F_1x02_P5.0mm_Vertical, F.Cu at (124.2, 46.4)
- added J29: Conn_01x05_Female, Connector_JST:JST_XH_B5B-XH-AM_1x05_P2.50mm_Vertical, F.Cu at (97.8, 123.8)
- added J3: Conn_01x03_Female, Connector_JST:JST_XH_B3B-XH-AM_1x03_P2.50mm_Vertical, F.Cu at (97.8, 64.8)
- added J30: Conn_01x05_Female, Connector_JST:JST_XH_B5B-XH-AM_1x05_P2.50mm_Vertical, F.Cu at (177.1, 104.2)
- added J31: Conn_01x07_Female, Connector_JST:JST_XH_B7B-XH-AM_1x07_P2.50mm_Vertical, F.Cu at (97.8, 104.8)
- added J32: Conn_01x07_Female, Connector_JST:JST_XH_B7B-XH-AM_1x07_P2.50mm_Vertical, F.Cu at (177.2, 113.3)
- added J4: Conn_01x05_Female, Connector_JST:JST_XH_B5B-XH-AM_1x05_P2.50mm_Vertical, F.Cu at (177.4, 135.9)
- added J5: Conn_01x05_Female, Connector_JST:JST_XH_B5B-XH-AM_1x05_P2.50mm_Vertical, F.Cu at (97.8, 71.8)
- added J6: Conn_01x07_Female, Connector_JST:JST_XH_B7B-XH-AM_1x07_P2.50mm_Vertical, F.Cu at (97.8, 130.9)
- added J7: Conn_01x07_Female, Connector_JST:JST_XH_B7B-XH-AM_1x07_P2.50mm_Vertical, F.Cu at (97.8, 78.9)
- added J8: XT30_F, Connector_AMASS:AMASS_XT30U-F_1x02_P5.0mm_Vertical, F.Cu at (148.2, 80.7)
- added J9: XT60_F, Connector_AMASS:AMASS_XT60-F_1x02_P7.20mm_Vertical, F.Cu at (145.8, 129.0)
Other:
- copper layers 0 -> 2
