File: lipo_parallel_board/lipo_parallel_board.kicad_pcb (KiCad board)
At the start: 2 copper layers, 32 parts, among them J1 Conn_01x07_Female, J10 Conn_01x03_Female, J11 Conn_01x03_Female, J12 XT30_F, J13 XT60_F, J14 XT30_F, J15 XT60_F, J16 Conn_01x05_Female, J17 Conn_01x05_Female, J18 XT30_F, J19 XT60_F, J2 Conn_01x03_Female, J20 XT30_F, J21 XT60_F, J22 Conn_01x07_Female, J23 Conn_01x07_Female, J24 XT30_F, J25 XT60_F, J26 Conn_01x03_Female, J27 Conn_01x03_Female, J28 XT30_F, J29 Conn_01x05_Female, J3 Conn_01x03_Female, J30 Conn_01x05_Female, J31 Conn_01x07_Female, J32 Conn_01x07_Female, J4 Conn_01x05_Female, J5 Conn_01x05_Female, J6 Conn_01x07_Female, J7 Conn_01x07_Female, J8 XT30_F, J9 XT60_F

Commit message: posizionato
Parts:
- moved J1 37.8 mm to (104.0, 55.4)
- moved J22 27.0 mm to (154.6, 130.9)
- moved J4 25.9 mm to (154.6, 123.8)
- moved J2 25.7 mm to (154.6, 116.7)
- moved J32 24.2 mm to (154.6, 104.8)
- moved J11 23.7 mm to (154.6, 90.7)
- moved J30 23.5 mm to (154.6, 97.8)
- moved J23 22.4 mm to (154.6, 78.8)
- moved J10 21.9 mm to (154.6, 64.4)
- moved J16 21.6 mm to (154.6, 71.6)
- moved J28 16.1 mm to (137.0, 56.2)
- moved J9 13.0 mm to (136.2, 120.2)
- moved J24 12.8 mm to (139.9, 130.2)
- moved J19 9.55 mm to (135.5, 68.2)
- moved J8 9.55 mm to (139.2, 77.6)
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
Commit message: terminato il master
Parts:
- added H1: MountingHole, MountingHole:MountingHole_3.2mm_M3, F.Cu at (98.0, 139.0)
- added H2: MountingHole, MountingHole:MountingHole_3.2mm_M3, F.Cu at (169.0, 139.0)
- added H3: MountingHole, MountingHole:MountingHole_3.2mm_M3, F.Cu at (98.0, 45.0)
- added H4: MountingHole, MountingHole:MountingHole_3.2mm_M3, F.Cu at (169.0, 45.0)
- J28: value XT30_F -> XT60_F; footprint Connector_AMASS:AMASS_XT30U-F_1x02_P5.0mm_Vertical -> Connector_AMASS:AMASS_XT60-F_1x02_P7.20mm_Vertical
- moved J28 8.16 mm to (128.8, 56.1)
- moved J1 5.00 mm to (99.2, 54.1)
- moved J12 2.00 mm to (122.7, 130.2)
- moved J13 2.00 mm to (119.0, 120.2)
- moved J14 2.00 mm to (122.7, 104.8)
- moved J18 2.00 mm to (122.7, 77.6)
- moved J21 2.00 mm to (119.0, 94.7)
- moved J25 2.00 mm to (119.0, 68.2)
Routing:
- net Net-(J1-Pad7): track 0.00 -> 225.0 mm, vias 0 -> 2
- net Net-(J1-Pad6): track 0.00 -> 223.3 mm, vias 0 -> 2
- net Net-(J1-Pad5): track 0.00 -> 221.5 mm, vias 0 -> 2
- net Net-(J1-Pad4): track 0.00 -> 218.5 mm, vias 0 -> 2
- net Net-(J1-Pad3): track 0.00 -> 216.7 mm, vias 0 -> 2
- net Net-(J1-Pad2): track 0.00 -> 214.1 mm, vias 0 -> 2
- net Net-(J1-Pad1): track 0.00 -> 212.2 mm, vias 0 -> 2
- net Net-(J12-Pad1): track 0.00 -> 194.4 mm
- net Net-(J12-Pad2): track 0.00 -> 174.8 mm
Other:
- board outline added: 79 x 102 mm
