File: lipo_parallel_board/lipo_parallel_board.kicad_sch (KiCad schematic)
At the start: 32 parts, among them J1 Conn_01x07_Female, J10 Conn_01x03_Female, J11 Conn_01x03_Female, J12 XT30_F, J13 XT60_F, J14 XT30_F, J15 XT60_F, J16 Conn_01x05_Female, J17 Conn_01x05_Female, J18 XT30_F, J19 XT60_F, J2 Conn_01x03_Female, J20 XT30_F, J21 XT60_F, J22 Conn_01x07_Female, J23 Conn_01x07_Female, J24 XT30_F, J25 XT60_F, J26 Conn_01x03_Female, J27 Conn_01x03_Female, J28 XT30_F, J29 Conn_01x05_Female, J3 Conn_01x03_Female, J30 Conn_01x05_Female, J31 Conn_01x07_Female, J32 Conn_01x07_Female, J4 Conn_01x05_Female, J5 Conn_01x05_Female, J6 Conn_01x07_Female, J7 Conn_01x07_Female, J8 XT30_F, J9 XT60_F

Commit message: posizionato
Parts:
- J28: value XT30_F -> XT60_F; footprint Connector_AMASS:AMASS_XT30U-F_1x02_P5.0mm_Vertical -> Connector_AMASS:AMASS_XT60-F_1x02_P7.20mm_Vertical
Changed lines of the file:
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@@
-(kicad_sch (version 20210406) (generator eeschema)
+(kicad_sch (version 20210606) (generator eeschema)
   (paper "A4")
   (junction (at 60.96 64.77) (diameter 1.016) (color 0 0 0 0))
@@
     (in_bom yes) (on_board yes)
     (property "Reference" "J28" (id 0) (at 168.7576 180.4204 0))
-    (property "Value" "XT30_F" (id 1) (at 163.6776 175.5817 0))
-    (property "Footprint" "Connector_AMASS:AMASS_XT30U-F_1x02_P5.0mm_Vertical" (id 2) (at 166.37 179.07 0)
+    (property "Value" "XT60_F" (id 1) (at 163.6776 175.5817 0))
+    (property "Footprint" "Connector_AMASS:AMASS_XT60-F_1x02_P7.20mm_Vertical" (id 2) (at 166.37 179.07 0)
       (effects (font (size 1.27 1.27)) hide)
     )
@@
     )
     (path "/b1cfcff2-c4b4-4394-a857-9695f4470d58"
-      (reference "J28") (unit 1) (value "XT30_F") (footprint "Connector_AMASS:AMASS_XT30U-F_1x02_P5.0mm_Vertical")
+      (reference "J28") (unit 1) (value "XT60_F") (footprint "Connector_AMASS:AMASS_XT60-F_1x02_P7.20mm_Vertical")
     )
     (path "/57c16db1-0054-4508-80a0-bc21684ad401"
