File: lipo_parallel_board/_autosave-lipo_parallel_board.kicad_sch (KiCad schematic)
At the start: 36 parts, among them J1 Conn_01x07_Female, J10 Conn_01x03_Female, J11 Conn_01x03_Female, J12 XT30_F, J13 XT60_F, J14 XT30_F, J15 XT60_F, J16 Conn_01x05_Female, J17 Conn_01x05_Female, J18 XT30_F, J19 XT60_F, J2 Conn_01x03_Female, J20 XT30_F, J21 XT60_F, J22 Conn_01x07_Female, J23 Conn_01x07_Female, J24 XT30_F, J25 XT60_F, J26 Conn_01x03_Female, J27 Conn_01x03_Female, J28 XT60_F, J29 Conn_01x05_Female, J3 Conn_01x03_Female, J30 Conn_01x05_Female, J31 Conn_01x07_Female, J32 Conn_01x07_Female, J4 Conn_01x05_Female, J5 Conn_01x05_Female, J6 Conn_01x07_Female, J7 Conn_01x07_Female, J8 XT30_F, J9 XT60_F

Commit message: terminato il master
Parts:
- gave numbers to parts that had none: 4
Changed lines of the file:
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@@
   (symbol (lib_id "Mechanical:MountingHole") (at 43.18 172.72 0) (unit 1)
     (in_bom yes) (on_board yes) (fields_autoplaced)
-    (property "Reference" "H?" (id 0) (at 45.7201 171.9591 0)
+    (property "Reference" "H1" (id 0) (at 45.7201 171.9591 0)
       (effects (font (size 1.27 1.27)) (justify left))
     )
@@
   (symbol (lib_id "Mechanical:MountingHole") (at 46.2411 185.916 0) (unit 1)
     (in_bom yes) (on_board yes) (fields_autoplaced)
-    (property "Reference" "H?" (id 0) (at 48.7812 185.1551 0)
+    (property "Reference" "H2" (id 0) (at 48.7812 185.1551 0)
       (effects (font (size 1.27 1.27)) (justify left))
     )
@@
   (symbol (lib_id "Mechanical:MountingHole") (at 66.4123 173.4573 0) (unit 1)
     (in_bom yes) (on_board yes) (fields_autoplaced)
-    (property "Reference" "H?" (id 0) (at 68.9524 172.6964 0)
+    (property "Reference" "H3" (id 0) (at 68.9524 172.6964 0)
       (effects (font (size 1.27 1.27)) (justify left))
     )
@@
   (symbol (lib_id "Mechanical:MountingHole") (at 67.31 185.42 0) (unit 1)
     (in_bom yes) (on_board yes) (fields_autoplaced)
-    (property "Reference" "H?" (id 0) (at 69.8501 184.6591 0)
+    (property "Reference" "H4" (id 0) (at 69.8501 184.6591 0)
       (effects (font (size 1.27 1.27)) (justify left))
     )
@@
   )
   (symbol_instances
+    (path "/d7696b1b-2485-4424-8b6d-e83abf8e561b"
+      (reference "H1") (unit 1) (value "MountingHole") (footprint "MountingHole:MountingHole_3.2mm_M3")
+    )
+    (path "/b7bd8ea1-99b7-44cb-a5f2-e732b37bcd13"
+      (reference "H2") (unit 1) (value "MountingHole") (footprint "MountingHole:MountingHole_3.2mm_M3")
+    )
     (path "/27f81133-e52b-4bdd-a058-31f02d46ce3b"
-      (reference "H?") (unit 1) (value "MountingHole") (footprint "MountingHole:MountingHole_3.2mm_M3")
+      (reference "H3") (unit 1) (value "MountingHole") (footprint "MountingHole:MountingHole_3.2mm_M3")
     )
     (path "/9885dae3-bb60-47cd-8cf9-fa88df541124"
-      (reference "H?") (unit 1) (value "MountingHole") (footprint "MountingHole:MountingHole_3.2mm_M3")
-    )
-    (path "/b7bd8ea1-99b7-44cb-a5f2-e732b37bcd13"
-      (reference "H?") (unit 1) (value "MountingHole") (footprint "MountingHole:MountingHole_3.2mm_M3")
-    )
-    (path "/d7696b1b-2485-4424-8b6d-e83abf8e561b"
-      (reference "H?") (unit 1) (value "MountingHole") (footprint "MountingHole:MountingHole_3.2mm_M3")
+      (reference "H4") (unit 1) (value "MountingHole") (footprint "MountingHole:MountingHole_3.2mm_M3")
     )
     (path "/d45b566e-41c0-4bd6-8494-ad1f3b06dbcf"
